Commit message: rufous work

File: src/dyse-robots/rufous_description/urdf/multirotor_base.xacro (robot description, xacro)
@@ -66,5 +66,5 @@
     <!-- attach multirotor_base_plugin to the base_link -->
 <!--     <gazebo>
-      <plugin filename="librofous_gazebo_plugins.so" name="rofous_gazebo_plugins">
+      <plugin filename="librufous_gazebo_plugins.so" name="rufous_gazebo_plugins">
         <robotNamespace>${robot_namespace}</robotNamespace>
         <linkName>${robot_namespace}/base_link</linkName>
@@ -106,5 +106,5 @@
           </xacro:if>
           <xacro:unless value="${use_own_mesh}">
-            <mesh filename="package://rofous_description/meshes/propeller_${direction}.dae"
+            <mesh filename="package://rufous_description/meshes/propeller_${direction}.dae"
               scale="${radius_rotor} ${radius_rotor} ${radius_rotor}" /> <!-- The propeller meshes have a radius of 1m -->
             <!-- <box size="${2*radius_rotor} 0.01 0.005"/> -->
